File: smart-lcc.kicad_pcb (KiCad board)
At the start: 2 copper layers, 59.5 x 53.2 mm, 16 parts, among them J1 USB_B_Micro, J10 Conn_01x04_Pin, J11 USB_B_Micro, J7 F0503-ZV-24-20T-R, J8 J-Link RP2040, J9 J-Link ESP32-S3, SW1 SW_DIP_x02, SW2 SW_SPDT, SW3 SW_Push, SW4 SW_Push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

Commit message: Updated with value for R2 resistor
Parts:
- R2: value R_Small -> 680R
Changed lines of the file:
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@@
         (effects (font (size 1 1) (thickness 0.15)))
     )
-    (fp_text value "R_Small" (at 3.81 1.92) (layer "F.Fab")
+    (fp_text value "680R" (at 3.81 1.92) (layer "F.Fab")
         (effects (font (size 1 1) (thickness 0.15)))
     )
