File: smart-lcc.kicad_sch (KiCad schematic)
At the start: 16 parts, among them J1 USB_B_Micro, J10 Conn_01x04_Pin, J11 USB_B_Micro, J7 F0503-ZV-24-20T-R, J8 J-Link RP2040, J9 J-Link ESP32-S3, SW1 SW_DIP_x02, SW2 SW_SPDT, SW3 SW_Push, SW4 SW_Push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

Commit message: Added manufacturing data
Parts:
- C5, C6, J10, J8, J9, R2, R7, SW1, SW2, SW3, SW4, SW5, U1: now left out of the parts list
Changed lines of the file:
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@@
   )
   (symbol (lib_id "Switch:SW_Push") (at 114.3 215.9 0) (unit 1)
-    (in_bom yes) (on_board yes) (dnp no)
+    (in_bom no) (on_board yes) (dnp no)
     (property "Reference" "SW4" (at 114.3 208.661 0)
       (effects (font (size 1.27 1.27)))
@@
   )
   (symbol (lib_id "Switch:SW_SPDT") (at 187.96 213.36 0) (unit 1)
-    (in_bom yes) (on_board yes) (dnp no) (fields_autoplaced)
+    (in_bom no) (on_board yes) (dnp no) (fields_autoplaced)
     (property "Reference" "SW2" (at 187.96 205.74 0)
       (effects (font (size 1.27 1.27)))
@@
   )
   (symbol (lib_id "Device:R_Small") (at 36.83 223.52 0) (unit 1)
-    (in_bom yes) (on_board yes) (dnp no) (fields_autoplaced)
+    (in_bom no) (on_board yes) (dnp no) (fields_autoplaced)
     (property "Reference" "R2" (at 39.37 222.25 0)
       (effects (font (size 1.27 1.27)) (justify left))
@@
   )
   (symbol (lib_id "Switch:SW_Push") (at 96.52 215.9 0) (unit 1)
-    (in_bom yes) (on_board yes) (dnp no)
+    (in_bom no) (on_board yes) (dnp no)
     (property "Reference" "SW3" (at 96.52 208.661 0)
       (effects (font (size 1.27 1.27)))
@@
   )
   (symbol (lib_id "Connector_Generic:Conn_02x10_Odd_Even") (at 46.99 292.1 0) (unit 1)
-    (in_bom yes) (on_board yes) (dnp no) (fields_autoplaced)
+    (in_bom no) (on_board yes) (dnp no) (fields_autoplaced)
     (property "Reference" "J8" (at 48.26 275.59 0)
       (effects (font (size 1.27 1.27)))
@@
   )
   (symbol (lib_id "Switch:SW_Push") (at 132.08 215.9 0) (unit 1)
-    (in_bom yes) (on_board yes) (dnp no)
+    (in_bom no) (on_board yes) (dnp no)
     (property "Reference" "SW5" (at 132.08 208.661 0)
       (effects (font (size 1.27 1.27)))
@@
   )
   (symbol (lib_id "Switch:SW_DIP_x02") (at 163.83 215.9 0) (unit 1)
-    (in_bom yes) (on_board yes) (dnp no) (fields_autoplaced)
+    (in_bom no) (on_board yes) (dnp no) (fields_autoplaced)
     (property "Reference" "SW1" (at 163.83 205.74 0)
       (effects (font (size 1.27 1.27)))
@@
   )
   (symbol (lib_id "Converter_DCDC:PTN78000H_EUS-5") (at 120.65 279.4 0) (unit 1)
-    (in_bom yes) (on_board yes) (dnp no) (fields_autoplaced)
+    (in_bom no) (on_board yes) (dnp no) (fields_autoplaced)
     (property "Reference" "U1" (at 120.65 269.24 0)
       (effects (font (size 1.27 1.27)))
@@
   )
   (symbol (lib_id "Device:C_Polarized_Small") (at 99.06 284.48 0) (unit 1)
-    (in_bom yes) (on_board yes) (dnp no) (fields_autoplaced)
+    (in_bom no) (on_board yes) (dnp no) (fields_autoplaced)
     (property "Reference" "C6" (at 101.6 282.6639 0)
       (effects (font (size 1.27 1.27)) (justify left))
@@
   )
   (symbol (lib_id "Device:R_Small") (at 133.35 284.48 0) (unit 1)
-    (in_bom yes) (on_board yes) (dnp no) (fields_autoplaced)
+    (in_bom no) (on_board yes) (dnp no) (fields_autoplaced)
     (property "Reference" "R7" (at 135.89 283.21 0)
       (effects (font (size 1.27 1.27)) (justify left))
@@
   )
   (symbol (lib_id "Connector_Generic:Conn_02x10_Odd_Even") (at 45.72 336.55 0) (unit 1)
-    (in_bom yes) (on_board yes) (dnp no) (fields_autoplaced)
+    (in_bom no) (on_board yes) (dnp no) (fields_autoplaced)
     (property "Reference" "J9" (at 46.99 320.04 0)
       (effects (font (size 1.27 1.27)))
@@
   )
   (symbol (lib_id "Connector:Conn_01x04_Pin") (at 157.48 328.93 0) (unit 1)
-    (in_bom yes) (on_board yes) (dnp no) (fields_autoplaced)
+    (in_bom no) (on_board yes) (dnp no) (fields_autoplaced)
     (property "Reference" "J10" (at 158.115 321.31 0)
       (effects (font (size 1.27 1.27)))
@@
   )
   (symbol (lib_id "Device:C_Polarized_Small") (at 140.97 284.48 0) (unit 1)
-    (in_bom yes) (on_board yes) (dnp no) (fields_autoplaced)
+    (in_bom no) (on_board yes) (dnp no) (fields_autoplaced)
     (property "Reference" "C5" (at 143.51 282.6639 0)
       (effects (font (size 1.27 1.27)) (justify left))

Commit message: Updated with value for R2 resistor
Parts:
- R2: value R_Small -> 680R
Changed lines of the file:
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@@
       (effects (font (size 1.27 1.27)) (justify left))
     )
-    (property "Value" "R_Small" (at 39.37 224.79 0)
+    (property "Value" "680R" (at 39.37 224.79 0)
       (effects (font (size 1.27 1.27)) (justify left))
     )
